Commit message: Simulation works with minimum plugin and  motor model with unmodified params

File: rotors_description/urdf/multirotor_base.xacro (robot description, xacro)
@@ -47,8 +47,8 @@
       </inertial>
       <visual>
-        <origin xyz="0 0 0" rpy="0 0 0" />
+        <origin xyz="0 0 0" rpy="1.5707963 0 3.1415926" />
         <geometry>
           <xacro:if value="${use_mesh_file}">
-            <mesh filename="${mesh_file}" scale="1 1 1" />
+            <mesh filename="${mesh_file}" scale="0.001 0.001 0.001" />
           </xacro:if>
           <xacro:unless value="${use_mesh_file}">
@@ -65,5 +65,5 @@
     </link>
     <!-- attach multirotor_base_plugin to the base_link -->
-    <gazebo>
+    <!-- <gazebo>
       <plugin filename="librotors_gazebo_multirotor_base_plugin.so" name="multirotor_base_plugin">
         <robotNamespace>${robot_namespace}</robotNamespace>
@@ -71,5 +71,5 @@
         <rotorVelocitySlowdownSim>${rotor_velocity_slowdown_sim}</rotorVelocitySlowdownSim>
       </plugin>
-    </gazebo>
+    </gazebo> -->
   </xacro:macro>
   <!-- Rotor joint and link -->
