Commit message: add the head and communication with yigle_ws

File: rotors_description/urdf/arm_test_nofakelink.xacro (robot description, xacro)
@@ -15,15 +15,13 @@
 <xacro:property name="friction" value="1e-5" />
 <!-- <xacro:property name="damping" value="5e-3" /> -->
-<xacro:property name="damping" value="5e-3" />
-  <gazebo reference="Link_shoulder_right">
+<xacro:property name="damping" value="2e-1" />
+  <!-- <gazebo reference="Link_shoulder_right">
     <mu1>0.2</mu1>
     <mu2>0.2</mu2>
   </gazebo>
-  <!-- Link2 -->
   <gazebo reference="Link_one_right">
     <mu1>0.2</mu1>
     <mu2>0.2</mu2>
   </gazebo>
-  <!-- Link3 -->
   <gazebo reference="Link_two_right">
     <mu1>0.2</mu1>
@@ -37,5 +35,5 @@
     <mu1>0.2</mu1>
     <mu2>0.2</mu2>
-  </gazebo>
+  </gazebo> -->
 <material name="blue">
     <color rgba="0 0 0.8 1"/>
@@ -87,5 +85,5 @@
 	<parent link="fixed_frame"/>
 	<child link="base_link_right"/>
-	<origin rpy="0 0 0" xyz="0.11475 0 0.009"/>
+	<origin rpy="0 0 0" xyz="-0.11475 0 0.009"/>
 </joint>
 <link name="base_link_right">
@@ -95,5 +93,4 @@
 		<mesh filename="package://rotors_description/meshes/arm/base_link.stl" scale="0.001 0.001 0.001"/>
 		</geometry>
-		<material name = "yellow"/>
 	</visual>
     <collision>
@@ -103,5 +100,5 @@
       </geometry>
     </collision>
-    <!-- <inertial>
+    <inertial>
       <origin xyz="-2.2068363e-3 -9.1832072e-6 3.1955704e-3" rpy="-0.1729 0 1.5708"/>
       <mass value="0.396"/>
@@ -110,25 +107,9 @@
         iyy="8.1358422e-4" iyz="0.0"
         izz="9.0317049e-4"/>
-    </inertial> -->
-    <!-- <inertial>
-      <origin xyz="-2.2068363e-3 0 3.1955704e-3" rpy="0 0 0"/>
-      <mass value="0.396"/>
-      <inertia
-        ixx="8.1358422e-4" ixy="0.0" ixz="0.0"
-        iyy="3.1455842e-4" iyz="0.0"
-        izz="9.0317049e-4"/>
-    </inertial> -->
-    <inertial>
-      <origin xyz="-2.2068363e-3 0 3.1955704e-3" rpy="0 0 0"/>
-      <mass value="0.396"/>
-      <inertia
-        ixx="8.1358422e-4" ixy="0.0" ixz="0.0"
-        iyy="3.1455842e-4" iyz="0.0"
-        izz="9.0317049e-4"/>
-    </inertial>
-</link>
- <joint name="Joint_shoulder_right" type="continuous">
+    </inertial>
+</link>
+ <joint name="Joint_shoulder_right" type="revolute">
  	<axis xyz="0 0 1"/>
- 	<!-- <limit effort="1000.0" lower="-3.14" upper="+3.14" velocity="1"/> -->
+ 	<limit effort="1000.0" lower="-3.14" upper="+3.14" velocity="1"/>
 	<parent link="base_link_right"/>
 	<child link="Link_shoulder_right"/>
@@ -142,19 +123,12 @@
 		<mesh filename="package://rotors_description/meshes/arm/j0.stl" scale="0.001 0.001 0.001"/>
 		</geometry>
-		<material name = "green"/>
-	</visual>
-    <collision>
-      <origin xyz="0 0 4.5368422e-3" rpy="0 0 0"/>
-      <geometry>
-        <box size="${width} 189e-3 189e-3"/>
-      </geometry>
-    </collision>
-    <!-- <collision>
-      <origin xyz="0 0 42.5e-3" rpy="0 0 0"/>
+	</visual>
+    <collision>
+      <origin xyz="0 0 42.572e-3" rpy="0 0 0"/>
       <geometry>
         <box size="41e-3 42.5e-3 85.144e-3"/>
       </geometry>
-    </collision> -->
-    <!-- <inertial>
+    </collision>
+    <inertial>
       <origin xyz="-3.0707866e-6 9.0724801e-5 3.3368422e-3" rpy="1.5790 -0.0021 1.7506"/>
       <mass value="1.586"/>
@@ -163,28 +137,12 @@
         iyy="5.8598889e-3" iyz="0.0"
         izz="6.2755829e-3"/>
-    </inertial> -->
-    <!-- <inertial>
-      <origin xyz="0 0 3.3368422e-3" rpy="0 0 0"/>
-      <mass value="1.586"/>
-      <inertia
-        ixx="6.2755829e-3" ixy="0.0" ixz="0.0"
-        iyy="9.7058009e-4" iyz="0.0"
-        izz="5.8598889e-3"/>
-    </inertial> -->
-    <inertial>
-      <origin xyz="0 0 4.5368422e-3" rpy="0 0 0"/>
-      <mass value="1.586"/>
-        <inertia
-	  ixx="${1.586 / 12.0 * (189e-3*189e-3 + 189e-3*189e-3)}" ixy="0.0" ixz="0.0"
-	  iyy="${1.586 / 12.0 * (width*width + 189e-3*189e-3)}" iyz="0.0"
-	  izz="${1.586 / 12.0 * (width*width + 189e-3*189e-3)}"/>
-    </inertial>
-</link>
-<joint name="Joint_1_right" type="continuous">
+    </inertial>
+</link>
+<joint name="Joint_1_right" type="revolute">
 	<axis xyz="1 0 0"/>
- 	<!-- <limit effort="1000.0" lower="0" upper="1.571" velocity="1"/> -->
+ 	<limit effort="1000.0" lower="0" upper="1.571" velocity="1"/>
 	<parent link="Link_shoulder_right"/>
 	<child link="Link_one_right"/>
-	<origin xyz="${width} 0 85.144e-3"/>
+	<origin xyz="0 0 85.144e-3"/>
   <dynamics damping="${damping}" friction="${friction}"/>
 </joint>
@@ -195,13 +153,12 @@
 		<mesh filename="package://rotors_description/meshes/arm/j1.stl" scale="0.001 0.001 0.001"/>
 		</geometry>
-		<material name = "black"/>
 	</visual>
     <collision>
       <origin xyz="0 0 56.5e-3" rpy="0 0 0"/>
       <geometry>
-        <box size="${width} ${width} 161e-3"/>
-      </geometry>
-    </collision>
-    <!-- <inertial>
+        <box size="41e-3 42.5e-3 113e-3"/>
+      </geometry>
+    </collision>
+    <inertial>
       <origin xyz="3.9623762e-4 5.2904518e-4 5.6046387e-2" rpy="-0.0193 -1.4555 -1.4511"/>
       <mass value="0.139"/>
@@ -210,28 +167,12 @@
         iyy="1.7117076e-4" iyz="0.0"
         izz="1.7370141e-4"/>
-    </inertial> -->
-    <!-- <inertial>
-      <origin xyz="0 0 5.6046387e-2" rpy=" 0 0 0"/>
-      <mass value="0.139"/>
-      <inertia
-        ixx="1.7117076e-4" ixy="0.0" ixz="0.0"
-        iyy="1.7370141e-4" iyz="0.0"
-        izz="5.7544276e-5"/>
-    </inertial> -->
-    <inertial>
-      <origin xyz="0 0 5.65e-2" rpy=" 0 0 0"/>
-      <mass value="0.139"/>
-        <inertia
-	  ixx="${0.139 / 12.0 * (width*width + 161e-3*161e-3)}" ixy="0.0" ixz="0.0"
-	  iyy="${0.139 / 12.0 * (161e-3*161e-3 + width*width)}" iyz="0.0"
-	  izz="${0.139 / 12.0 * (width*width + width*width)}"/>
-    </inertial>
-</link>
-<joint name="Joint_2_right" type="continuous">
+    </inertial>
+</link>
+<joint name="Joint_2_right" type="revolute">
 	<axis xyz="1 0 0"/>
- 	<!-- <limit effort="1000.0" lower="-1.571" upper="0" velocity="1"/> -->
+ 	<limit effort="1000.0" lower="-1.571" upper="0" velocity="1"/>
 	<parent link="Link_one_right"/>
 	<child link="Link_two_right"/>
-	<origin xyz="-${width} 0 0.113"/>
+	<origin xyz="0 0 0.113"/>
   <dynamics damping="${damping}" friction="${friction}"/>
 </joint>
@@ -242,13 +183,12 @@
 		<mesh filename="package://rotors_description/meshes/arm/j2.stl" scale="0.001 0.001 0.001"/>
 		</geometry>
-		<material name = "red"/>
 	</visual>
     <collision>
       <origin xyz="0 0 69e-3" rpy="0 0 0"/>
       <geometry>
-        <box size="${width} ${width} 186e-3"/>
-      </geometry>
-    </collision>
-    <!-- <inertial>
+        <box size="41e-3 42.5e-3 138e-3"/>
+      </geometry>
+    </collision>
+    <inertial>
       <origin xyz="5.1358654e-4 1.4848633e-3 6.4707125e-2" rpy="3.0686 -1.5089 1.6549"/>
       <mass value="0.154"/>
@@ -257,28 +197,12 @@
         iyy="2.7365867e-4" iyz="0.0"
         izz="2.7990892e-4"/>
-    </inertial> -->
-    <!-- <inertial>
-      <origin xyz="0 1.4848633e-3 6.4707125e-2" rpy="0 0 0"/>
-      <mass value="0.154"/>
-      <inertia
-        ixx="2.7365867e-4" ixy="0.0" ixz="0.0"
-        iyy="2.7990892e-4" iyz="0.0"
-        izz="9.2363919e-5"/>
-    </inertial> -->
-        <inertial>
-      <origin xyz="0 0 6.9e-2" rpy="0 0 0"/>
-      <mass value="0.154"/>
-        <inertia
-	  ixx="${0.154 / 12.0 * (width*width + 186e-3*186e-3)}" ixy="0.0" ixz="0.0"
-	  iyy="${0.154 / 12.0 * (186e-3*186e-3 + width*width)}" iyz="0.0"
-	  izz="${0.154 / 12.0 * (width*width + width*width)}"/>
-    </inertial>
-</link>
-<joint name="Joint_3_right" type="continuous">
+    </inertial>
+</link>
+<joint name="Joint_3_right" type="revolute">
 	<axis xyz="1 0 0"/>
- 	<!-- <limit effort="1000.0" lower="0" upper="1.571" velocity="1"/> -->
+ 	<limit effort="1000.0" lower="0" upper="1.571" velocity="1"/>
 	<parent link="Link_two_right"/>
 	<child link="Link_three_right"/>
-	<origin xyz="${width} 0 0.138"/>
+	<origin xyz="0 0 0.138"/>
   <dynamics damping="${damping}" friction="${friction}"/>
 </joint>
@@ -289,13 +213,12 @@
 		<mesh filename="package://rotors_description/meshes/arm/j3.stl" scale="0.001 0.001 0.001"/>
 		</geometry>
-		<material name = "blue"/>
 	</visual>
     <collision>
       <origin xyz="0 0 75.1e-3" rpy="0 0 0"/>
       <geometry>
-        <box size="${width}  ${width}  175e-3"/>
-      </geometry>
-    </collision>
-    <!-- <inertial>
+        <box size="41e-3 42.5e-3 150.2e-3"/>
+      </geometry>
+    </collision>
+    <inertial>
       <origin xyz="1.0689991e-4 4.5539723e-3 8.0348105e-2" rpy="0.0503 -1.4936 -1.6299"/>
       <mass value="0.207"/>
@@ -304,25 +227,9 @@
         iyy="3.4408597e-4" iyz="0.0"
         izz="3.6490830e-4"/>
-    </inertial> -->
-    <!-- <inertial>
-      <origin xyz="0 4.5539723e-3 8.0348105e-2" rpy="0 0 0"/>
-      <mass value="0.207"/>
-      <inertia
-        ixx="3.4408597e-4" ixy="0.0" ixz="0.0"
-        iyy="3.6490830e-4" iyz="0.0"
-        izz="8.4188171e-5"/>
-    </inertial> -->
-    <inertial>
-      <origin xyz="0 0 63e-3" rpy="0 0 0"/>
-      <mass value="0.207"/>
-        <inertia
-	  ixx="${0.207 / 12.0 * (width*width + 175e-3*175e-3)}" ixy="0.0" ixz="0.0"
-	  iyy="${0.207 / 12.0 * (175e-3*175e-3 + width*width)}" iyz="0.0"
-	  izz="${0.207 / 12.0 * (width*width + width*width)}"/>
-    </inertial>
-</link>
-<joint name="Joint_wrist_right" type="continuous">
+    </inertial>
+</link>
+<joint name="Joint_wrist_right" type="revolute">
 	<axis xyz="0 0 1"/>
- 	<!-- <limit effort="1000.0" lower="-3.14" upper="3.14" velocity="1"/> -->
+ 	<limit effort="1000.0" lower="-3.14" upper="3.14" velocity="1"/>
 	<parent link="Link_three_right"/>
 	<child link="Link_hand_right"/>
@@ -336,5 +243,4 @@
     <mesh filename="package://rotors_description/meshes/arm/hand.stl" scale="0.001 0.001 0.001"/>
     </geometry>
-		<material name = "black"/>
 	</visual>
     <collision>
@@ -344,5 +250,5 @@
       </geometry>
     </collision>
-    <!-- <inertial>
+    <inertial>
       <origin xyz="-5.1914952e-3 9.4338844e-4 8.4791871e-2" rpy="2.7807 -1.4896 1.8174"/>
       <mass value="0.505"/>
@@ -351,205 +257,6 @@
         iyy="1.1324016e-3" iyz="0.0"
         izz="1.3591446e-3"/>
-    </inertial> -->
-    <!-- <inertial>
-      <origin xyz="-5.1914952e-3 9.4338844e-4 8.4791871e-2" rpy="0 0 0"/>
-      <mass value="0.505"/>
-      <inertia
-        ixx="1.1324016e-3" ixy="0.0" ixz="0.0"
-        iyy="1.3591446e-3" iyz="0.0"
-        izz="3.2734333e-4 "/>
-    </inertial> -->
-    <inertial>
-      <origin xyz="0 0 102.5e-3" rpy="0 0 0"/>
-      <mass value="0.505"/>
-        <inertia
-	  ixx="${0.505 / 12.0 * (width*width + 205e-3*205e-3)}" ixy="0.0" ixz="0.0"
-	  iyy="${0.505 / 12.0 * (205e-3*205e-3+ width*width)}" iyz="0.0"
-	  izz="${0.505 / 12.0 * (width*width + width*width)}"/>
-    </inertial>
-</link>
-<!-- <joint name="fixed_joint_left" type="fixed">
-	<parent link="fixed_frame"/>
-	<child link="base_link_left"/>
-	<origin rpy="0 0 0" xyz="-0.11475 0 0.009"/>
-</joint>
-<link name="base_link_left">
-	<visual>
-		<origin rpy="0 0 0" xyz="0 0 0"/>
-		<geometry>
-		<mesh filename="package://rotors_description/meshes/arm/base_link.stl" scale="0.001 0.001 0.001"/>
-		</geometry>
-		<material name = "yellow"/>
-	</visual>
-    <collision>
-      <origin xyz="0 0 39.875e-3" rpy="0 0 0"/>
-      <geometry>
-        <cylinder radius="26.05e-3" length="79.75e-3"/>
-      </geometry>
-    </collision>
-    <inertial>
-      <origin xyz="-2.2068363e-3 -9.1832072e-6 3.1955704e-3" rpy="-0.1729 0 1.5708"/>
-      <mass value="0.396"/>
-      <inertia
-        ixx="3.1455842e-4" ixy="0.0" ixz="0.0"
-        iyy="8.1358422e-4" iyz="0.0"
-        izz="9.0317049e-4"/>
-    </inertial>
-</link>
- <joint name="Joint_shoulder_left" type="continuous">
- 	<axis xyz="0 0 1"/>
- 	<limit effort="1000.0" lower="-3.14" upper="+3.14" velocity="1"/>
-	<parent link="base_link_left"/>
-	<child link="Link_shoulder_left"/>
-	<origin xyz="0 0 79.75e-3"/>
-  <dynamics damping="${damping}" friction="${friction}"/>
-</joint>
-<link name="Link_shoulder_left">
-	<visual>
-		<origin rpy="0 0 0" xyz="0 0 0"/>
-		<geometry>
-		<mesh filename="package://rotors_description/meshes/arm/j0.stl" scale="0.001 0.001 0.001"/>
-		</geometry>
-		<material name = "green"/>
-	</visual>
-    <collision>
-      <origin xyz="0 0 42.572e-3" rpy="0 0 0"/>
-      <geometry>
-        <box size="41e-3 42.5e-3 85.144e-3"/>
-      </geometry>
-    </collision>
-    <inertial>
-      <origin xyz="-3.0707866e-6 9.0724801e-5 3.3368422e-3" rpy="1.5790 -0.0021 1.7506"/>
-      <mass value="1.586"/>
-      <inertia
-        ixx="9.7058009e-4" ixy="0.0" ixz="0.0"
-        iyy="5.8598889e-3" iyz="0.0"
-        izz="6.2755829e-3"/>
-    </inertial>
-</link>
-<joint name="Joint_1_left" type="continuous">
-	<axis xyz="1 0 0"/>
- 	<limit effort="1000.0" lower="0" upper="1.571" velocity="1"/>
-	<parent link="Link_shoulder_left"/>
-	<child link="Link_one_left"/>
-	<origin xyz="0 0 85.144e-3"/>
-  <dynamics damping="${damping}" friction="${friction}"/>
-</joint>
-<link name="Link_one_left">
-	<visual>
-		<origin rpy="0 0 0" xyz="0 0 24e-3"/>
-		<geometry>
-		<mesh filename="package://rotors_description/meshes/arm/j1.stl" scale="0.001 0.001 0.001"/>
-		</geometry>
-		<material name = "black"/>
-	</visual>
-    <collision>
-      <origin xyz="0 0 56.5e-3" rpy="0 0 0"/>
-      <geometry>
-        <box size="41e-3 42.5e-3 113e-3"/>
-      </geometry>
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
File: rotors_description/urdf/neck_head_test.xacro (robot description, xacro)
@@ -1,135 +1,147 @@
 <?xml version="1.0"?>
-<robot xmlns:xacro="http://ros.org/wiki/xacro">
-<xacro:macro name="neck_head_macro"
-  params="robot_namespace parent_link">
+<robot name="head_test" xmlns:xacro="http://ros.org/wiki/xacro">
+<!-- <xacro:macro name="neck_head_macro"
+  params="robot_namespace parent_link"> -->
 <gazebo>
   <plugin name="gazebo_ros_control" filename="libgazebo_ros_control.so">
-    <robotNamespace>${robot_namespace}</robotNamespace>
+    <robotNamespace>/head_test</robotNamespace>
   </plugin>
 </gazebo>
-<xacro:property name="PI" value="3.1415926535897931"/>
-<joint name="DJI_leg_joint" type="fixed">
-	<parent link="${parent_link}"/>
-	<child link="DJI_leg_link"/>
-	<origin rpy="${PI} 0 0" xyz="0 y z"/>
-</joint>
-<link name="DJI_leg_link">
-	<visual>
-		<origin rpy="0 0 0" xyz="0 0 0"/>
-		<geometry>
-		<mesh filename="" scale="0.001 0.001 0.001"/>
-		</geometry>
-	</visual>
-    <collision>
-      <origin xyz="0 0 0" rpy="0 0 0"/>
-      <geometry>
-      </geometry>
-    </collision>
-    <inertial>
-      <origin xyz="0 0 0" rpy="0 0 0"/>
-      <mass value="0"/>
-      <inertia
-        ixx="" ixy="0.0" ixz="0.0"
-        iyy="" iyz="0.0"
-        izz=""/>
+<link name="world">
+</link>
+<joint name="DJI_connect_joint" type="fixed">
+	<parent link="world"/>
+	<child link="DJI_connect_link"/>
+	<origin rpy="${pi+0.0873} 0 0" xyz="0 -74.58e-3 1"/>
+</joint>
+<link name="DJI_connect_link">
+	<visual>
+      <origin xyz="0 79e-3 13.5e-3" rpy="0 0 0"/>
+      <geometry>
+	      <box size="80e-3 158e-3 27e-3"/>
+      </geometry>
+	</visual>
+    <collision>
+      <origin xyz="0 79e-3 13.5e-3" rpy="0 0 0"/>
+      <geometry>
+	      <box size="80e-3 158e-3 27e-3"/>
+      </geometry>
+    </collision>
+    <inertial>
+      <origin xyz="0 81.25e-3 13.5e-3" rpy="0 0 0"/>
+      <mass value="0.05"/>
+      <inertia
+        ixx="${0.05/12*(158e-3*158e-3+27e-3*27e-3)}" ixy="0.0" ixz="0.0"
+        iyy="${0.05/12*(27e-3*27e-3+80e-3*80e-3)}" iyz="0.0"
+        izz="${0.05/12*(158e-3*158e-3+80e-3*80e-3)}"/>
     </inertial>
 </link>
 <joint name="neck_base_joint" type="fixed">
-	<parent link="DJI_leg_link"/>
+	<parent link="DJI_connect_link"/>
 	<child link="neck_base_link"/>
-	<origin rpy="0 0 0" xyz="0 y z"/>
+	<origin rpy="0 0 0" xyz="0 117e-3 27e-3"/>
 </joint>
 <link name="neck_base_link">
 	<visual>
-		<origin rpy="0 0 0" xyz="0 0 0"/>
-		<geometry>
-		<mesh filename="" scale="0.001 0.001 0.001"/>
-		</geometry>
-	</visual>
-    <collision>
-      <origin xyz="0 0 0" rpy="0 0 0"/>
-      <geometry>
-      </geometry>
-    </collision>
-    <inertial>
-      <origin xyz="0 0 0" rpy="0 0 0"/>
-      <mass value="0"/>
-      <inertia
-        ixx="" ixy="0.0" ixz="0.0"
-        iyy="" iyz="0.0"
-        izz=""/>
-    </inertial>
-</link>
-<joint name="neck_joint_1" type="fixed">
+      <origin xyz="0 0 40e-3" rpy="0 0 0"/>
+      <geometry>
+        <box size="80e-3 80e-3 80e-3"/>
+      </geometry>
+	</visual>
+    <collision>
+      <origin xyz="0 0 40e-3" rpy="0 0 0"/>
+      <geometry>
+        <box size="80e-3 80e-3 80e-3"/>
+      </geometry>
+    </collision>
+    <inertial>
+      <origin xyz="-1.6749134e-05 1.3880927e-3 3.2904335e-2" rpy="-0.3776 -0.0858 1.5403"/>
+      <mass value="0.454"/>
+      <inertia
+        ixx="1.6874028e-4" ixy="0.0" ixz="0.0"
+        iyy="1.7773673e-4" iyz="0.0"
+        izz="1.8020647e-4"/>
+    </inertial>
+</link>
+<joint name="neck_joint_1" type="revolute">
+ 	<axis xyz="0 1 0"/>
+ 	<limit effort="1000.0" lower="${-pi}" upper="${pi}" velocity="1"/>
 	<parent link="neck_base_link"/>
 	<child link="neck_link_1"/>
-	<origin rpy="0 0 0" xyz="0 y z"/>
+	<origin rpy="0 0 0" xyz="0 45.5e-3 34e-3"/>
+  <dynamics damping="1e-5" friction="1e-5"/>
 </joint>
 <link name="neck_link_1">
 	<visual>
-		<origin rpy="0 0 0" xyz="0 0 0"/>
-		<geometry>
-		<mesh filename="" scale="0.001 0.001 0.001"/>
-		</geometry>
-	</visual>
-    <collision>
-      <origin xyz="0 0 0" rpy="0 0 0"/>
-      <geometry>
-      </geometry>
-    </collision>
-    <inertial>
-      <origin xyz="0 0 0" rpy="0 0 0"/>
-      <mass value="0"/>
-      <inertia
-        ixx="" ixy="0.0" ixz="0.0"
-        iyy="" iyz="0.0"
-        izz=""/>
-    </inertial>
-</link>
-<joint name="neck_joint_2" type="fixed">
+      <origin xyz="0 -2.75e-3 0" rpy="0 0 0"/>
+      <geometry>
+        <box size="80e-3 5.5e-3 80e-3"/>
+      </geometry>
+	</visual>
+    <collision>
+      <origin xyz="0 -2.75e-3 0" rpy="0 0 0"/>
+      <geometry>
+        <box size="80e-3 5.5e-3 80e-3"/>
+      </geometry>
+    </collision>
+    <inertial>
+      <origin xyz="7.3157519e-3 2.6015782e-2 0" rpy="0 0 0.5020"/>
+      <mass value="0.0866"/>
+      <inertia
+        ixx="6.8361134e-5" ixy="0.0" ixz="0.0"
+        iyy="1.1299140e-4" iyz="0.0"
+        izz="1.3810438e-4"/>
+    </inertial>
+</link>
+<joint name="neck_joint_2" type="revolute">
+ 	<axis xyz="1 0 0"/>
+ 	<limit effort="1000.0" lower="${-pi/2}" upper="${pi/2}" velocity="1"/>
 	<parent link="neck_link_1"/>
 	<child link="head_link"/>
-	<origin rpy="${PI} 0 0" xyz="0 y z"/>
+	<origin rpy="0 0 0" xyz="0 56e-3 0"/>
+  <dynamics damping="1e-5" friction="1e-5"/>
 </joint>
 <link name="head_link">
 	<visual>
-		<origin rpy="0 0 0" xyz="0 0 0"/>
-		<geometry>
-		<mesh filename="" scale="0.001 0.001 0.001"/>
-		</geometry>
-	</visual>
-    <collision>
-      <origin xyz="0 0 0" rpy="0 0 0"/>
-      <geometry>
-      </geometry>
-    </collision>
-    <inertial>
-      <origin xyz="0 0 0" rpy="0 0 0"/>
-      <mass value="0"/>
-      <inertia
-        ixx="" ixy="0.0" ixz="0.0"
-        iyy="" iyz="0.0"
-        izz=""/>
-    </inertial>
-</link>
+      <origin xyz="0 40e-3 0" rpy="0 0 0"/>
+      <geometry>
+        <sphere radius="60e-3"/>
+      </geometry>
+	</visual>
+    <collision>
+      <origin xyz="0 40e-3 0" rpy="0 0 0"/>
+      <geometry>
+        <sphere radius="60e-3"/>
+      </geometry>
+    </collision>
+    <inertial>
+      <origin xyz="1.6724729e-04 2.5974293e-2 1.6809604e-2" rpy="1.5708 -0.0334 0"/>
+      <mass value="0.95"/>
+      <inertia
+        ixx="1.4514462e-3" ixy="0.0" ixz="0.0"
+        iyy="2.0518578e-3" iyz="0.0"
+        izz="2.1893905e-3"/>
+    </inertial>
+</link>
+ <xacro:property name="camera_link" value="0.05" /> <!-- Size of square 'camera' box -->
 <joint name="eye_joint" type="fixed">
+  <axis xyz="0 1 0" />
 	<parent link="head_link"/>
 	<child link="left_camera_frame"/>
-	<origin rpy="0 0 ${PI/2}" xyz="0 y z"/>
+	<origin rpy="${-pi/2} ${-pi/2} 0" xyz="31e-3 46.83e-3 81.95e-3"/>
 </joint>
   <!-- Camera -->
   <link name="left_camera_frame">
     <collision>
-      <origin xyz="0 0 0" rpy="0 0 0"/>
-      <geometry>
-	<box size="${camera_link} ${camera_link} ${camera_link}"/>
+      <origin xyz="-15.25e-3 -31e-3 0 " rpy="0 0 0"/>
+      <geometry>
+	      <box size="30.5e-3 124.5e-3 26.5e-3 "/>
       </geometry>
     </collision>
     <visual>
-      <origin xyz="0 0 0" rpy="0 0 0"/>
-      <geometry>
-	<box size="${camera_link} ${camera_link} ${camera_link}"/>
-      </geometry>
-      <material name="red"/>
+      <origin xyz=" -15.25e-3 -31e-3 0" rpy="0 0 0"/>
+      <geometry>
+	      <box size="30.5e-3 124.5e-3 26.5e-3"/>
+      </geometry>
     </visual>
     <inertial>
@@ -171,5 +183,5 @@
       </camera>
       <camera name="right">
-        <pose>0 -0.07 0 0 0 0</pose>
+        <pose>0 -0.060 0 0 0 0</pose>
         <horizontal_fov>1.3962634</horizontal_fov>
         <image>
@@ -225,4 +237,4 @@
     </actuator>
   </transmission>
-</xacro:macro>
+<!-- </xacro:macro>  -->
 </robot>

File: rotors_description/urdf/yigle.xacro (robot description, xacro)
@@ -49,4 +49,5 @@
   <xacro:include filename="$(find rotors_description)/urdf/multirotor_base.xacro" />
   <xacro:include filename="$(find rotors_description)/urdf/arm_base.xacro" />
+  <xacro:include filename="$(find rotors_description)/urdf/head_base.xacro" />
   <!-- Instantiate multirotor_base_macro once -->
   <xacro:multirotor_base_macro
@@ -189,3 +190,6 @@
     parent_link="${namespace}/base_link">
   </xacro:arm_base_macro>
+  <xacro:neck_head_macro
+    parent_link="${namespace}/base_link">
+  </xacro:neck_head_macro>
 </robot>
