Commit message: backup after successful simulation

File: rotors_description/urdf/arm_base.xacro (robot description, xacro)
@@ -164,5 +164,5 @@
 	<parent link="Link_three_right"/>
 	<child link="Link_hand_right"/>
-	<origin xyz="0 0 0.1502"/>
+	<origin xyz="0 0 0.1502" rpy="0 0 ${pi/2}"/>
   <dynamics damping="${damping}" friction="${friction}"/>
 </joint>
@@ -171,11 +171,37 @@
 		<origin rpy="0 0 0 " xyz="0 0 0"/>
 		<geometry>
-    <mesh filename="package://rotors_description/meshes/arm/hand.stl" scale="0.001 0.001 0.001"/>
+    <mesh filename="package://rotors_description/meshes/arm/hand_right.stl" scale="0.001 0.001 0.001"/>
     </geometry>
 	</visual>
     <collision>
+      <surface>
+            <!-- <contact>
+              <ode>
+                <max_vel>10</max_vel>
+                <min_depth>0.001</min_depth>
+              </ode>
+            </contact>         -->
+        <friction>
+          <ode>
+            <mu>5</mu>
+            <mu2>5</mu2>
+            <kp value="10000000.0" />
+			      <kd value="1.0" />
+          </ode>
+        </friction>
+        <!-- <soft_contact>
+          <dart>
+            <bone_attachment>100
+            </bone_attachment>
+            <stiffness>100
+            </stiffness>
+            <damping>10
+            </damping>
+          </dart>
+        </soft_contact> -->
+      </surface>
       <origin xyz="0 0 102.556e-3" rpy="0 0 0"/>
       <geometry>
-        <box size="41e-3 54e-3 205.122e-3"/>
+        <box size="80e-3 36e-3 205.122e-3"/>
       </geometry>
     </collision>
@@ -341,5 +367,5 @@
 	<parent link="Link_three_left"/>
 	<child link="Link_hand_left"/>
-	<origin xyz="0 0 0.1502"/>
+	<origin xyz="0 0 0.1502" rpy="0 0 ${-pi/2}"/>
   <dynamics damping="${damping}" friction="${friction}"/>
 </joint>
@@ -348,11 +374,31 @@
 		<origin rpy="0 0 0 " xyz="0 0 0"/>
 		<geometry>
-    <mesh filename="package://rotors_description/meshes/arm/hand.stl" scale="0.001 0.001 0.001"/>
+    <mesh filename="package://rotors_description/meshes/arm/hand_left.stl" scale="0.001 0.001 0.001"/>
     </geometry>
 	</visual>
     <collision>
+      <surface>
+        <friction>
+          <ode>
+            <mu>5</mu>
+            <mu2>5</mu2>
+            			<kp value="10000000.0" />
+			<kd value="1.0" />
+          </ode>
+        </friction>
+        <!-- <soft_contact>
+          <dart>
+            <bone_attachment>100
+            </bone_attachment>
+            <stiffness>100
+            </stiffness>
+            <damping>10
+            </damping>
+          </dart>
+        </soft_contact> -->
+      </surface>
       <origin xyz="0 0 102.556e-3" rpy="0 0 0"/>
       <geometry>
-        <box size="41e-3 54e-3 205.122e-3"/>
+        <box size="80e-3 36e-3 205.122e-3"/>
       </geometry>
     </collision>

File: rotors_description/urdf/arm_base_fakelink.xacro (robot description, xacro)
@@ -246,5 +246,5 @@
 		<origin rpy="0 0 0 " xyz="0 0 0"/>
 		<geometry>
-    <mesh filename="package://rotors_description/meshes/arm/hand.stl" scale="0.001 0.001 0.001"/>
+    <mesh filename="package://rotors_description/meshes/arm/hand_right.stl" scale="0.001 0.001 0.001"/>
     </geometry>
 		<material name = "black"/>
@@ -481,5 +481,5 @@
 		<origin rpy="0 0 0 " xyz="0 0 0"/>
 		<geometry>
-    <mesh filename="package://rotors_description/meshes/arm/hand.stl" scale="0.001 0.001 0.001"/>
+    <mesh filename="package://rotors_description/meshes/arm/hand_left.stl" scale="0.001 0.001 0.001"/>
     </geometry>
 		<material name = "black"/>

File: rotors_description/urdf/arm_test_nofakelink copy.xacro (robot description, xacro)
@@ -332,5 +332,5 @@
 		<origin rpy="0 0 0 " xyz="0 0 0"/>
 		<geometry>
-    <mesh filename="package://rotors_description/meshes/arm/hand.stl" scale="0.001 0.001 0.001"/>
+    <mesh filename="package://rotors_description/meshes/arm/hand_right.stl" scale="0.001 0.001 0.001"/>
     </geometry>
 		<material name = "black"/>
@@ -531,5 +531,5 @@
 		<origin rpy="0 0 0 " xyz="0 0 0"/>
 		<geometry>
-    <mesh filename="package://rotors_description/meshes/arm/hand.stl" scale="0.001 0.001 0.001"/>
+    <mesh filename="package://rotors_description/meshes/arm/hand_left.stl" scale="0.001 0.001 0.001"/>
     </geometry>
 		<material name = "black"/>

File: rotors_description/urdf/arm_test_nofakelink.xacro (robot description, xacro)
@@ -241,5 +241,5 @@
 		<origin rpy="0 0 0 " xyz="0 0 0"/>
 		<geometry>
-    <mesh filename="package://rotors_description/meshes/arm/hand.stl" scale="0.001 0.001 0.001"/>
+    <mesh filename="package://rotors_description/meshes/arm/hand_right.stl" scale="0.001 0.001 0.001"/>
     </geometry>
 	</visual>

File: rotors_description/urdf/head_base.xacro (robot description, xacro)
@@ -170,6 +170,6 @@
         <horizontal_fov>1.3962634</horizontal_fov>
         <image>
-          <width>800</width>
-          <height>800</height>
+          <width>1280</width>
+          <height>720</height>
           <format>R8G8B8</format>
         </image>
@@ -185,9 +185,9 @@
       </camera>
       <camera name="right">
-        <pose>0 -0.060 0 0 0 0</pose>
+        <pose>0 -0.070 0 0 0 0</pose>
         <horizontal_fov>1.3962634</horizontal_fov>
         <image>
-          <width>800</width>
-          <height>800</height>
+          <width>1280</width>
+          <height>720</height>
           <format>R8G8B8</format>
         </image>
@@ -205,5 +205,5 @@
         <alwaysOn>true</alwaysOn>
         <updateRate>0.0</updateRate>
-        <cameraName>multisense_sl/camera</cameraName>
+        <cameraName>camera</cameraName>
         <imageTopicName>image_raw</imageTopicName>
         <cameraInfoTopicName>camera_info</cameraInfoTopicName>

File: rotors_description/urdf/multirotor_base.xacro (robot description, xacro)
@@ -47,5 +47,5 @@
       </inertial>
       <visual>
-        <origin xyz="0 0 0" rpy="1.5707963 0 3.1415926" />
+        <origin xyz="0 0 0" rpy="${pi} 0 0" />
         <geometry>
           <xacro:if value="${use_mesh_file}">

File: rotors_description/urdf/neck_head_test.xacro (robot description, xacro)
@@ -168,6 +168,6 @@
         <horizontal_fov>1.3962634</horizontal_fov>
         <image>
-          <width>800</width>
-          <height>800</height>
+          <width>1280</width>
+          <height>720</height>
           <format>R8G8B8</format>
         </image>
@@ -183,9 +183,9 @@
       </camera>
       <camera name="right">
-        <pose>0 -0.060 0 0 0 0</pose>
+        <pose>0 -0.070 0 0 0 0</pose>
         <horizontal_fov>1.3962634</horizontal_fov>
         <image>
-          <width>800</width>
-          <height>800</height>
+          <width>1280</width>
+          <height>720</height>
           <format>R8G8B8</format>
         </image>
@@ -203,5 +203,5 @@
         <alwaysOn>true</alwaysOn>
         <updateRate>0.0</updateRate>
-        <cameraName>multisense_sl/camera</cameraName>
+        <cameraName>yigle/camera</cameraName>
         <imageTopicName>image_raw</imageTopicName>
         <cameraInfoTopicName>camera_info</cameraInfoTopicName>

File: rotors_description/urdf/yigle.xacro (robot description, xacro)
@@ -24,8 +24,8 @@
   <xacro:property name="mass" value="9.5" /> <!-- [kg] -->
   <xacro:property name="body_width" value="1.5" /> <!-- TODO: [m] -->
-  <xacro:property name="body_height" value="1.0" /> <!-- TODO: [m] -->
+  <xacro:property name="body_height" value="0.3" /> <!-- TODO: [m] -->
   <xacro:property name="mass_rotor" value="0.005" /> <!-- [kg] -->
   <xacro:property name="arm_length" value="0.567" /> <!-- [m] -->
-  <xacro:property name="rotor_offset_top" value="0.14" /> <!-- TODO: [m] -->
+  <xacro:property name="rotor_offset_top" value="0.13" /> <!-- TODO: [m] -->
   <xacro:property name="radius_rotor" value="0.1" /> <!-- [m] -->
   <xacro:property name="motor_constant" value="8.54858e-06" /> <!-- [kg m/s^2] -->
