Commit message: add arm urdf, self-designed actuator, gazebo-ros-control actuator, and test code for arm, lee controller for  drone and arm drone together

File: rotors_description/urdf/component_snippets.xacro (robot description, xacro)
@@ -17,4 +17,29 @@
 -->
 <robot xmlns:xacro="http://ros.org/wiki/xacro">
+  <xacro:macro name="arm_actuator_plugin_macro"
+    params="namespace">
+    <gazebo>
+      <plugin name="arm_actuator_interface" filename="librotors_gazebo_arm_actuator_interface.so">
+        <robotNamespace>${namespace}</robotNamespace>
+      </plugin>
+    </gazebo>
+  </xacro:macro>
+  <xacro:macro name="arm_actuator_plugin_macro_nofakelink"
+    params="namespace">
+    <gazebo>
+      <plugin name="arm_actuator_interface_nofakelink" filename="librotors_gazebo_arm_actuator_interface_nofakelink.so">
+        <robotNamespace>${namespace}</robotNamespace>
+        <!-- <gazebo_joint_control_pid>
+          <p>0.01</p>
+          <i>0.0001</i>
+          <d>0.0001</d>
+          <iMax>0</iMax>
+          <iMin>0</iMin>
+          <cmdMax>0.15</cmdMax>
+          <cmdMin>-0.15</cmdMin>
+        </gazebo_joint_control_pid> -->
+      </plugin>
+    </gazebo>
+  </xacro:macro>
   <!-- Macro to add logging to a bag file. -->
   <xacro:macro name="bag_plugin_macro"

File: rotors_description/urdf/yigle.xacro (robot description, xacro)
@@ -16,5 +16,5 @@
   limitations under the License.
 -->
-<robot name="firefly" xmlns:xacro="http://ros.org/wiki/xacro">
+<robot name="yigle" xmlns:xacro="http://ros.org/wiki/xacro">
   <!-- Properties -->
   <xacro:property name="namespace" value="$(arg namespace)" />
@@ -22,5 +22,5 @@
   <xacro:property name="use_mesh_file" value="true" />
   <xacro:property name="mesh_file" value="package://rotors_description/meshes/M600.stl" />
-  <xacro:property name="mass" value="1.5" /> <!-- [kg] -->
+  <xacro:property name="mass" value="9.5" /> <!-- [kg] -->
   <xacro:property name="body_width" value="1.5" /> <!-- TODO: [m] -->
   <xacro:property name="body_height" value="1.0" /> <!-- TODO: [m] -->
@@ -40,6 +40,6 @@
   <!-- Property Blocks -->
   <xacro:property name="body_inertia">
-    <inertia ixx="0.0347563" ixy="0.0" ixz="0.0" iyy="0.0458929" iyz="0.0" izz="0.0977" /> <!-- [kg m^2] [kg m^2] [kg m^2] [kg m^2] [kg m^2] [kg m^2] -->
-  </xacro:property>
+    <inertia ixx="6.8902275e-1" ixy="3.1406183e-04" ixz="-6.6251112e-04" iyy="6.5920645e-1" iyz="2.9107974e-04" izz="1.0416577" /> [kg m^2] [kg m^2] [kg m^2] [kg m^2] [kg m^2] [kg m^2]
+ </xacro:property>
   <!-- inertia of a single rotor, assuming it is a cuboid. Height=3mm, width=15mm -->
   <xacro:property name="rotor_inertia">
@@ -48,4 +48,5 @@
   <!-- Included URDF Files -->
   <xacro:include filename="$(find rotors_description)/urdf/multirotor_base.xacro" />
+  <xacro:include filename="$(find rotors_description)/urdf/arm_base.xacro" />
   <!-- Instantiate multirotor_base_macro once -->
   <xacro:multirotor_base_macro
@@ -184,3 +185,7 @@
     <xacro:insert_block name="rotor_inertia" />
   </xacro:vertical_rotor>
+  <xacro:arm_base_macro
+    robot_namespace="${namespace}"
+    parent_link="${namespace}/base_link">
+  </xacro:arm_base_macro>
 </robot>

File: rotors_description/urdf/yigle_base.xacro (robot description, xacro)
@@ -16,5 +16,5 @@
   limitations under the License.
 -->
-<robot name="firefly" xmlns:xacro="http://ros.org/wiki/xacro">
+<robot name="yigle" xmlns:xacro="http://ros.org/wiki/xacro">
   <xacro:include filename="$(find rotors_description)/urdf/component_snippets.xacro" />
   <!-- Instantiate firefly "mechanics" -->
