Commit message: reconstruct

File: rotors_description/urdf/multirotor_base.xacro (robot description, xacro)
@@ -1,4 +1,5 @@
 <?xml version="1.0"?>
 <!--
+  Modifications Copyright 2022 Fanyi Kong, NMMI, Italy
   Copyright 2015 Fadri Furrer, ASL, ETH Zurich, Switzerland
   Copyright 2015 Michael Burri, ASL, ETH Zurich, Switzerland
