Commit message: backup alot of things

File: aerial_ego_simulation/urdf/arm_base.xacro (robot description, xacro)
@@ -39,5 +39,5 @@
       <parent link="${parent_link}"/>
       <child link="base_link_right"/>
-      <origin rpy="0 ${PI} 0" xyz="-0.11475 0 0.009"/>
+      <origin rpy="0 ${PI} 0" xyz="-0.1135 0 -0.074"/>
     </joint>
     <link name="base_link_right">
@@ -224,5 +224,5 @@
       <parent link="${parent_link}"/>
       <child link="base_link_left"/>
-      <origin rpy="0 3.1416 0" xyz="0.11475 0 0.009"/>
+      <origin rpy="0 3.1416 0" xyz="0.1135 0 -0.074"/>
     </joint>
     <link name="base_link_left">
